Commit message: Added the different lidar configurations

File: src/catkin_ws/src/LMS1xx/urdf/sick_lms1xx.urdf.xacro (robot description, xacro)
@@ -28,6 +28,25 @@
   <!--<xacro:macro name="sick_lms1xx" params="frame:=laser topic:=scan sample_size:=720 update_rate:=50
                min_angle:=-2.35619 max_angle:=2.35619 min_range:=0.1 max_range:=30.0 robot_namespace:=/" >-->
+  <!-- Blind Spot -->
+  <!-- Robot 1 -->
+  <!--<xacro:macro name="sick_lms1xx" params="frame:=laser topic:=scan sample_size:=720 update_rate:=50
+               min_angle:=-1 max_angle:=1 min_range:=0.1 max_range:=5.0 robot_namespace:=/" > -->
+  <!-- Robot 2 -->
+    <!--<xacro:macro name="sick_lms1xx" params="frame:=laser topic:=scan sample_size:=720 update_rate:=50
+               min_angle:=-1.57 max_angle:=1.57 min_range:=0.1 max_range:=10.0 robot_namespace:=/" >-->
+  <!-- Distance robots -->
+  <!-- Robot 1 -->
   <xacro:macro name="sick_lms1xx" params="frame:=laser topic:=scan sample_size:=720 update_rate:=50
-               min_angle:=-1 max_angle:=1 min_range:=1 max_range:=30.0 robot_namespace:=/" >
+               min_angle:=-1.57 max_angle:=1.57 min_range:=0.1 max_range:=5.0 robot_namespace:=/" >
+  <!-- Robot 2 -->
+    <!--<xacro:macro name="sick_lms1xx" params="frame:=laser topic:=scan sample_size:=720 update_rate:=50
+               min_angle:=-1.57 max_angle:=1.57 min_range:=0.1 max_range:=10.0 robot_namespace:=/" >-->
+  <!-- Block size robots -->
+  <!-- Robot 1 -->
+  <!--<xacro:macro name="sick_lms1xx" params="frame:=laser topic:=scan sample_size:=32 update_rate:=50
+               min_angle:=-1.57 max_angle:=1.57 min_range:=0.1 max_range:=10.0 robot_namespace:=/" > -->
+  <!-- Robot 2 -->
+    <!--<xacro:macro name="sick_lms1xx" params="frame:=laser topic:=scan sample_size:=32 update_rate:=50
+               min_angle:=-1.57 max_angle:=1.57 min_range:=0.1 max_range:=10.0 robot_namespace:=/" >-->
     <link name="${frame}">
       <inertial>

Commit message: Added some readme files, added world files.

File: src/catkin_ws/src/LMS1xx/urdf/sick_lms1xx.urdf.xacro (robot description, xacro)
@@ -31,19 +31,19 @@
   <!-- Robot 1 -->
   <!--<xacro:macro name="sick_lms1xx" params="frame:=laser topic:=scan sample_size:=720 update_rate:=50
-               min_angle:=-1 max_angle:=1 min_range:=0.1 max_range:=5.0 robot_namespace:=/" > -->
+               min_angle:=-1 max_angle:=1 min_range:=0.1 max_range:=10.0 robot_namespace:=/" >-->
   <!-- Robot 2 -->
-    <!--<xacro:macro name="sick_lms1xx" params="frame:=laser topic:=scan sample_size:=720 update_rate:=50
-               min_angle:=-1.57 max_angle:=1.57 min_range:=0.1 max_range:=10.0 robot_namespace:=/" >-->
+  <xacro:macro name="sick_lms1xx" params="frame:=laser topic:=scan sample_size:=720 update_rate:=50
+               min_angle:=-1.57 max_angle:=1.57 min_range:=0.1 max_range:=10.0 robot_namespace:=/" >
   <!-- Distance robots -->
   <!-- Robot 1 -->
-  <xacro:macro name="sick_lms1xx" params="frame:=laser topic:=scan sample_size:=720 update_rate:=50
-               min_angle:=-1.57 max_angle:=1.57 min_range:=0.1 max_range:=5.0 robot_namespace:=/" >
+  <!--<xacro:macro name="sick_lms1xx" params="frame:=laser topic:=scan sample_size:=720 update_rate:=50
+               min_angle:=-1.57 max_angle:=1.57 min_range:=0.1 max_range:=5.0 robot_namespace:=/" >-->
   <!-- Robot 2 -->
-    <!--<xacro:macro name="sick_lms1xx" params="frame:=laser topic:=scan sample_size:=720 update_rate:=50
+  <!--<xacro:macro name="sick_lms1xx" params="frame:=laser topic:=scan sample_size:=720 update_rate:=50
                min_angle:=-1.57 max_angle:=1.57 min_range:=0.1 max_range:=10.0 robot_namespace:=/" >-->
   <!-- Block size robots -->
   <!-- Robot 1 -->
-  <!--<xacro:macro name="sick_lms1xx" params="frame:=laser topic:=scan sample_size:=32 update_rate:=50
-               min_angle:=-1.57 max_angle:=1.57 min_range:=0.1 max_range:=10.0 robot_namespace:=/" > -->
+  <!--<xacro:macro name="sick_lms1xx" params="frame:=laser topic:=scan sample_size:=16 update_rate:=50
+               min_angle:=-1.57 max_angle:=1.57 min_range:=0.1 max_range:=10.0 robot_namespace:=/" >-->
   <!-- Robot 2 -->
     <!--<xacro:macro name="sick_lms1xx" params="frame:=laser topic:=scan sample_size:=32 update_rate:=50
